Commit message: horde of specific task files

File: assets/cylinder/heldout/obj_1.urdf (robot description, URDF)
Before this commit: robot object, 1 links, 0 joints
Links:
- link object: mass 0.050894 -> 0.059828; geometry collision cylinder length=0.045000 radius=0.046000; visual cylinder length=0.045000 radius=0.046000

File: assets/cylinder/train/obj_2.urdf (robot description, URDF)
Before this commit: robot object, 1 links, 0 joints
Links:
- link object: mass 0.030411 -> 0.040351; geometry collision cylinder length=0.095000 radius=0.026000; visual cylinder length=0.095000 radius=0.026000

File: assets/sphere/heldout/obj_0.urdf (robot description, URDF)
Before this commit: robot object, 1 links, 0 joints
Links:
- link object: mass 0.076341 -> 0.044179; geometry collision sphere radius=0.037500; visual sphere radius=0.037500

File: assets/sphere/train/obj_0.urdf (robot description, URDF)
Before this commit: robot object, 1 links, 0 joints
Links:
- link object: mass 0.027452 -> 0.039086; geometry collision sphere radius=0.036000; visual sphere radius=0.036000

File: assets/sphere/train/obj_1.urdf (robot description, URDF)
Before this commit: robot object, 1 links, 0 joints
Links:
- link object: mass 0.053617 -> 0.049695; geometry collision sphere radius=0.039000; visual sphere radius=0.039000
